File: technische tekeningen/elektronisch/planB/10102025/10102025.kicad_sch (KiCad schematic)
At the start: 6 parts, among them M1 Motor_DC, M2 Motor_DC

Commit message: a
Parts:
- added SW1: Start, symbol Switch:SW_Push
Connections:
- net +3.3V is gone; now on net VCC_3.3V: 8channel-ir-sensor1. (VCC), ESP-WROOM-32-devkit1. (3.3V)
- net GND: now also SW1.2
- net VCC_3.3V: now reaches 8channel-ir-sensor1. (VCC)
- net GPIO21: now reaches DRV883-module1. (IN1)
- net GPIO21: now also ESP-WROOM-32-devkit1. (3.3V)
- new net: 8channel-ir-sensor1. (VCC), ESP-WROOM-32-devkit1. (3.3V) (x6)
- new net: BT1.1 (+), DRV883-module1. (IN1), ESP-WROOM-32-devkit1. (3.3V)
- new net: DRV883-module1. (IN1), ESP-WROOM-32-devkit1. (3.3V) (x2)
- new net: ESP-WROOM-32-devkit1. (3.3V), SW1.1
- new net GPIO19: DRV883-module1. (IN1), ESP-WROOM-32-devkit1. (3.3V)
Other:
- moved on the sheet: DRV883-module1, M1, M2

Commit message: com
Connections:
- new net: 8channel-ir-sensor1. (VCC), ESP-WROOM-32-devkit1. (3.3V) (x6)
- new net: BT1.1 (+), DRV883-module1. (IN1), ESP-WROOM-32-devkit1. (3.3V)
- new net: DRV883-module1. (IN1), ESP-WROOM-32-devkit1. (3.3V) (x2)
Other:
- moved on the sheet: 8channel-ir-sensor1, BT1, DRV883-module1, ESP-WROOM-32-devkit1, M1, M2, SW1
