File: technische tekeningen/elektronisch/planA/planA.kicad_sch (KiCad schematic)
At the start: 20 parts, among them J1 Connector_usb-serial, M1 Motor_DC, M2 Motor_DC, SW1 reset, U1 ESP32-S3-WROOM-1, U2 AMS1117-3.3

Commit message: update
Parts:
- removed J1: Connector_usb-serial, symbol Connector:Conn_01x04_Socket
- added D4: Wifi, LED_THT:LED_D5.0mm, symbol Device:LED
- added J1: Connector_usb_to_ttl, symbol Connector:Conn_01x06_Socket
- added R3: 75, Resistor_THT:R_Axial_DIN0204_L3.6mm_D1.6mm_P7.62mm_Horizontal, symbol Device:R
- added SW2: start/stop, Button_Switch_SMD:SW_SPST_PTS645Sx43SMTR92, symbol Switch:SW_Push
- D1: footprint (none) -> LED_THT:LED_D5.0mm
- R1, R2: footprint (none) -> Resistor_THT:R_Axial_DIN0204_L3.6mm_D1.6mm_P7.62mm_Horizontal
- SW1: footprint (none) -> Button_Switch_SMD:SW_SPST_PTS645Sx43SMTR92
Connections:
- net ESP_3.3V: now also J1.2 (Pin_2)
- net GND: now also D4.1 (K), J1.6 (Pin_6), SW2.1
- net RXD0: now also J1.4 (Pin_4)
- net TXD0: now also J1.3 (Pin_3)
- net at M2.1 (+): now also DRV-module1. (IN1)
- net at M2.2 (-): now also DRV-module1. (IN1)
- net at M1.1 (+): now also DRV-module1. (IN1)
- net at M1.2 (-): now also DRV-module1. (IN1)
- net GPIO17: now reaches U1.10 (GPIO17/U1TXD/ADC2_CH6)
- net GPIO17: now also DRV-module1. (IN1)
- net GPIO18: now reaches U1.11 (GPIO18/U1RXD/ADC2_CH7/CLK_OUT3)
- net GPIO18: now also DRV-module1. (IN1)
- net at U1.33 (MTDO/GPIO40/CLK_OUT2): now also SW2.2
- net at U1.35 (MTMS/GPIO42): now also R3.2
- new net: D4.2 (A), R3.1
Other:
- moved on the sheet: 8channel-ir-sensor1, C5, C6, D2, D3, DRV-module1, M1, M2, R2, SW1, U1

Commit message: begin pcb
Parts:
- removed C1, C3, C5: 10uF, symbol Device:C
- added C1, C3, C5: 10uF, Capacitor_THT:CP_Radial_D5.0mm_P2.00mm, symbol Device:C_Polarized
- added J2: jumper esp voltage, Connector_PinHeader_2.54mm:PinHeader_1x03_P2.54mm_Vertical, symbol Connector:Conn_01x03_Pin
- BT1: footprint (none) -> Connector_PinHeader_2.54mm:PinHeader_1x02_P2.54mm_Vertical
- C2, C4, C6: footprint (none) -> Capacitor_THT:C_Disc_D4.3mm_W1.9mm_P5.00mm
- D1: footprint LED_THT:LED_D5.0mm -> LED_THT:LED_D3.0mm
- D2, D3: footprint (none) -> Diode_THT:D_A-405_P7.62mm_Horizontal
- DRV1: renamed from DRV-module1; value ~ -> DRV8833 module; footprint (none) -> eigenfootprints:DRV8833_Module_1x06_P2,54mm
- J1: footprint (none) -> Connector_PinSocket_2.54mm:PinSocket_1x06_P2.54mm_Vertical
- M1, M2: footprint (none) -> eigenfootprints:motor holder
- R1, R3: value 75 -> 150(220); footprint Resistor_THT:R_Axial_DIN0204_L3.6mm_D1.6mm_P7.62mm_Horizontal -> Resistor_THT:R_Axial_DIN0207_L6.3mm_D2.5mm_P10.16mm_Horizontal
- R2: footprint Resistor_THT:R_Axial_DIN0204_L3.6mm_D1.6mm_P7.62mm_Horizontal -> Resistor_THT:R_Axial_DIN0207_L6.3mm_D2.5mm_P10.16mm_Horizontal
- SN1: renamed from 8channel-ir-sensor1; value ~ -> 8 channel ir sensor; footprint (none) -> eigenfootprints:8channel_ir_sensor_1x11_P2.54mm
- SW1, SW2: footprint Button_Switch_SMD:SW_SPST_PTS645Sx43SMTR92 -> Button_Switch_THT:SW_PUSH_6mm_H4.3mm
Connections:
- net ESP_3.3V: now also SN1.11 (VCC), SN1.2 (IR), C5.1, J2.2 (Pin_2); no longer C4.1, J1.2 (Pin_2), SN1. (VCC), U2.2 (VO)
- net GND: now also DRV1.3 (GND), SN1.1 (GND), C1.2, C3.2, C5.2; no longer DRV1. (IN1), SN1. (VCC)
- net GPIO17: now also DRV1.1 (IN4); no longer DRV1. (IN1)
- net GPIO18: now also DRV1.2 (IN3); no longer DRV1. (IN1)
- net GPIO45: now also DRV1.5 (IN2); no longer DRV1. (IN1)
- net GPIO46: now also DRV1.6 (IN1); no longer DRV1. (IN1)
- net RXD0: now also J1.3 (TX); no longer J1.4 (Pin_4)
- net TXD0: now also J1.2 (RX); no longer J1.3 (Pin_3)
- net at DRV1. (ULT): now also M1.2 (-)
- net at U1.12 (GPIO8/TOUCH8/ADC1_CH7/SUBSPICS1): now also SN1.5 (D3); no longer SN1. (VCC)
- net at U1.17 (GPIO9/TOUCH9/ADC1_CH8/FSPIHD/SUBSPIHD): now also SN1.4 (D2); no longer SN1. (VCC)
- net at U1.18 (GPIO10/TOUCH10/ADC1_CH9/FSPICS0/FSPIIO4/SUBSPICS0): now also SN1.3 (D1); no longer SN1. (VCC)
- net at U1.38 (GPIO2/TOUCH2/ADC1_CH1): now also SN1.10 (D8); no longer SN1. (VCC)
- net at U1.4 (GPIO4/TOUCH4/ADC1_CH3): now also SN1.9 (D7); no longer SN1. (VCC)
- net at U1.5 (GPIO5/TOUCH5/ADC1_CH4): now also SN1.8 (D6); no longer SN1. (VCC)
- net at U1.6 (GPIO6/TOUCH6/ADC1_CH5): now also SN1.7 (D5); no longer SN1. (VCC)
- net at U1.7 (GPIO7/TOUCH7/ADC1_CH6): now also SN1.6 (D4); no longer SN1. (VCC)
- net VCC_7.4V renamed BT_7.4V
- net BT_7.4V: now also DRV1.4 (VCC), C1.1; no longer DRV1. (IN1)
- new net: J1.4 (VCC), J2.3 (Pin_3)
- new net VCC_3.3V: C3.1, C4.1, J2.1 (Pin_1), U2.2 (VO)
Other:
- moved on the sheet: D1, R1

Commit message: pcb
Parts:
- removed D2, D3: D, Diode_THT:D_A-405_P7.62mm_Horizontal, symbol Device:D
- added C7: 0u1F, Capacitor_THT:C_Disc_D4.3mm_W1.9mm_P5.00mm, symbol Device:C
- added R4: 10k, Resistor_THT:R_Axial_DIN0207_L6.3mm_D2.5mm_P10.16mm_Horizontal, symbol Device:R
- added SW3: boot, Button_Switch_THT:SW_PUSH_6mm_H4.3mm, symbol Switch:SW_Push
Connections:
- net ESP_3.3V: now also R4.1
- net GND: now also C7.2, SW3.2
- net GPIO17: now also DRV1.2 (IN3); no longer DRV1.1 (IN4)
- net GPIO18: now also DRV1.1 (IN4); no longer DRV1.2 (IN3)
- net at R2.2, SW1.2: now also U1.3 (EN), C7.1
- net at DRV1. (ULT): now also M1.2 (-)
- net GPIO0: no longer names the net of U1.27 (GPIO0/BOOT)
- net GPIO0: now also R4.2, SW3.1
Other:
- moved on the sheet: C5, C6, D1, R1
