File: technische tekeningen/elektronisch/planA/planA.kicad_pcb (KiCad board)
At the start: 2 copper layers, 24 parts, among them J1 Connector_usb_to_ttl, J2 jumper esp voltage, M1 Motor_DC, M2 Motor_DC, SW1 reset, SW2 start/stop, U1 ESP32-S3-WROOM-1, U2 AMS1117-3.3

Commit message: pcb
Parts:
- removed D2, D3: D, Diode_THT:D_A-405_P7.62mm_Horizontal
- added Boot: boot, Button_Switch_THT:SW_PUSH_6mm_H4.3mm, F.Cu at (213.8, 104.8)
- added C7: 0u1F, Capacitor_THT:C_Disc_D4.3mm_W1.9mm_P5.00mm, F.Cu at (237.0, 107.0)
- added R4: 10k, Resistor_THT:R_Axial_DIN0207_L6.3mm_D2.5mm_P10.16mm_Horizontal, F.Cu at (241.4, 130.5)
- USB Vcc Bat.: renamed from J2
- moved SN1 55.7 mm to (187.0, 111.7)
- moved Power 43.0 mm to (232.0, 105.5)
- moved Start/Stop 35.8 mm to (224.2, 138.2)
- moved R3 33.1 mm to (241.4, 134.5), turned to 0 degrees
- moved J1 23.1 mm to (219.0, 70.5), turned to 0 degrees
- moved R1 10.8 mm to (244.0, 115.5), turned to 180 degrees
- moved USB Vcc Bat. 5.17 mm to (231.1, 59.5)
- moved DRV8833 2.41 mm to (243.1, 70.5)
- moved Reset 2.26 mm to (214.0, 93.5)
- moved R2 0.75 mm to (244.0, 112.0)
- renumbered BT1 to Battery, DRV1 to DRV8833, D1 to Power, SW1 to Reset, SW2 to Start/Stop, D4 to Wifi
Connections:
- DRV8833 pad 1: GPIO17 -> GPIO18
- DRV8833 pad 2: GPIO18 -> GPIO17
- R2 pad 2: Net-(D2-A) -> Net-(U1-EN)
- Reset pad 2: Net-(D2-A) -> Net-(U1-EN)
- U1 pad 27: GPIO0 -> Net-(U1-GPIO0/BOOT)
- U1 pad 3: Net-(D2-K) -> Net-(U1-EN)
Routing:
- net GND: track 108.0 -> 323.8 mm
- net Net-(SN1-D8): track 0.00 -> 138.1 mm
- net TXD0: track 0.00 -> 121.4 mm, vias 0 -> 1
- net RXD0: track 0.00 -> 117.9 mm, vias 0 -> 1
- net ESP_3.3V: track 81.8 -> 158.4 mm
- net Net-(U1-GPIO0/BOOT): track 0.00 -> 76.3 mm
- net Net-(SN1-D7): track 20.5 -> 87.7 mm
- net Net-(SN1-D6): track 18.9 -> 84.5 mm
- net Net-(SN1-D5): track 17.7 -> 81.4 mm
- net GPIO45: track 0.00 -> 62.1 mm, vias 0 -> 1
- net Net-(SN1-D4): track 16.5 -> 78.2 mm
- net Net-(SN1-D2): track 21.1 -> 82.4 mm
- net Net-(SN1-D3): track 12.6 -> 73.6 mm
- net Net-(SN1-D1): track 22.2 -> 82.3 mm
- net GPIO18: track 0.00 -> 55.2 mm, vias 0 -> 1
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Other:
- board outline added: 91.5 x 100 mm
- board text added: "3.3V"
- board text added: "ESP32-S3-WROOM-1"
- board text added: "GND"
- board text added: "Motor holder"
- board text added: "Rx"
- board text added: "Tx"

Commit message: d
Parts:
- moved USB Vcc Bat. 120.4 mm to (110.8, 53.2)
- moved Battery 120.4 mm to (147.8, 72.9)
- moved Boot 120.4 mm to (93.5, 98.4)
- moved C1 120.4 mm to (141.2, 78.7)
- moved C2 120.4 mm to (145.8, 77.2)
- moved C3 120.4 mm to (132.2, 78.7)
- moved C4 120.4 mm to (136.8, 77.2)
- moved C5 120.4 mm to (125.4, 99.9)
- moved C6 120.4 mm to (120.9, 100.9)
- moved C7 120.4 mm to (116.8, 100.7)
- moved DRV8833 120.4 mm to (122.9, 64.2)
- moved J1 120.4 mm to (98.8, 64.1)
- moved Power 120.4 mm to (111.8, 99.2)
- moved R1 120.4 mm to (123.8, 109.2)
- moved R2 120.4 mm to (123.8, 105.7)
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Routing:
- net GND: track 323.8 -> 348.9 mm
- net Net-(U1-GPIO0/BOOT): track 76.3 -> 80.0 mm
- net ESP_3.3V: track 158.4 -> 162.0 mm
- net BT_7.4V: track 45.3 -> 47.8 mm
- net GPIO18: track 55.2 -> 56.5 mm
- net RXD0: track 117.9 -> 119.1 mm
- net GPIO17: track 51.0 -> 52.0 mm
- net TXD0: track 121.4 -> 122.3 mm
- net Net-(SN1-D8): track 138.1 -> 138.9 mm
- net GPIO45: track 62.1 -> 62.7 mm
Other:
- board size 91.5 x 100 mm -> 103.5 x 100 mm
- board text added: "Line follwoing robot"
